Commit message: Sync actuator mass and hand limits

File: urdf/s2_v1_complex_clamp.urdf (robot description, URDF)
Before this commit: robot walker_s2_v1_complex_description, 35 links, 34 joints
Links:
- link L_hand_link: mass 0.28014837 -> 0.380120
- link R_hand_link: mass 0.28014837 -> 0.380120

File: urdf/s2_v1_complex_hand.urdf (robot description, URDF)
Before this commit: robot walker_s2_v1_complex_hand_description, 59 links, 58 joints
Links:
- link L_hand_base_link: mass 0 -> 0.169970
- link L_index_ip_link: mass 0.0133493 -> 0.01962738
- link L_index_mpp_link: mass 0.0147008 -> 0.02481999
- link L_little_ip_link: mass 0.0117927 -> 0.01658133
- link L_little_mpp_link: mass 0.0143021 -> 0.02481999
- link L_middle_ip_link: mass 0.0148881 -> 0.01962738
- link L_middle_mpp_link: mass 0.0143021 -> 0.02481999
- link L_palm_link: mass 0 -> 0.44979018
- link L_ring_ip_link: mass 0.0137479 -> 0.01962738
- link L_ring_mpp_link: mass 0.0143021 -> 0.02481999
- link L_thumb_cmp_link: mass 0.0151103 -> 0.01405089
- link L_thumb_ip_link: mass 0.0173112 -> 0.01901012
- link L_thumb_mpp_link: mass 0.067412 -> 0.09019498
- link R_hand_base_link: mass 0 -> 0.169970
- link R_index_ip_link: mass 0.0133493 -> 0.01962738
- link R_index_mpp_link: mass 0.0147008 -> 0.02481999
- link R_little_ip_link: mass 0.0117927 -> 0.01658133
- link R_little_mpp_link: mass 0.0143021 -> 0.02481999
- link R_middle_ip_link: mass 0.0148881 -> 0.01962738
- link R_middle_mpp_link: mass 0.0143021 -> 0.02481999
- link R_palm_link: mass 0 -> 0.44979018
- link R_ring_ip_link: mass 0.0137479 -> 0.01962738
- link R_ring_mpp_link: mass 0.0143021 -> 0.02481999
- link R_thumb_cmp_link: mass 0.0151103 -> 0.01405089
- link R_thumb_ip_link: mass 0.0173112 -> 0.01901012
- link R_thumb_mpp_link: mass 0.067412 -> 0.09019498
Joints:
- joint L_index_ip_joint: limit lower=0 upper=1.62 effort=0.311 velocity=0 -> lower=0 upper=1.62 effort=0.311 velocity=2.09
- joint L_index_mpp_joint: limit lower=0 upper=1.46 effort=0.583 velocity=0 -> lower=0 upper=1.6685 effort=0.583 velocity=2.09
- joint L_little_ip_joint: limit lower=0 upper=1.62 effort=0.257 velocity=0 -> lower=0 upper=1.62 effort=0.257 velocity=2.09
- joint L_little_mpp_joint: limit lower=0 upper=1.46 effort=0.528 velocity=0 -> lower=0 upper=1.6685 effort=0.528 velocity=2.09
- joint L_middle_ip_joint: limit lower=0 upper=1.62 effort=0.332 velocity=0 -> lower=0 upper=1.62 effort=0.332 velocity=2.09
- joint L_middle_mpp_joint: limit lower=0 upper=1.46 effort=0.604 velocity=0 -> lower=0 upper=1.6685 effort=0.604 velocity=2.09
- joint L_ring_ip_joint: limit lower=0 upper=1.62 effort=0.311 velocity=0 -> lower=0 upper=1.62 effort=0.311 velocity=2.09
- joint L_ring_mpp_joint: limit lower=0 upper=1.46 effort=0.583 velocity=0 -> lower=0 upper=1.6685 effort=0.583 velocity=2.09
- joint L_thumb_cmp_joint: limit lower=-0.96 upper=0 effort=0.704 velocity=0 -> lower=-0.96 upper=0 effort=0.704 velocity=2.09
- joint L_thumb_ip_joint: limit lower=0 upper=1.05 effort=0.182 velocity=0 -> lower=0 upper=1.05 effort=0.182 velocity=2.09
- joint L_thumb_mpp_joint: limit lower=0 upper=1.04 effort=0.632 velocity=0 -> lower=0 upper=1.04 effort=0.632 velocity=2.09
- joint R_index_ip_joint: limit lower=0 upper=1.62 effort=0.311 velocity=0 -> lower=0 upper=1.62 effort=0.311 velocity=2.09
- joint R_index_mpp_joint: limit lower=0 upper=1.46 effort=0.583 velocity=0 -> lower=0 upper=1.6685 effort=0.583 velocity=2.09
- joint R_little_ip_joint: limit lower=0 upper=1.62 effort=0.257 velocity=0 -> lower=0 upper=1.62 effort=0.257 velocity=2.09
- joint R_little_mpp_joint: limit lower=0 upper=1.46 effort=0.528 velocity=0 -> lower=0 upper=1.6685 effort=0.528 velocity=2.09
- joint R_middle_ip_joint: limit lower=0 upper=1.62 effort=0.332 velocity=0 -> lower=0 upper=1.62 effort=0.332 velocity=2.09
- joint R_middle_mpp_joint: limit lower=0 upper=1.46 effort=0.604 velocity=0 -> lower=0 upper=1.6685 effort=0.604 velocity=2.09
- joint R_ring_ip_joint: limit lower=0 upper=1.62 effort=0.311 velocity=0 -> lower=0 upper=1.62 effort=0.311 velocity=2.09
- joint R_ring_mpp_joint: limit lower=0 upper=1.46 effort=0.583 velocity=0 -> lower=0 upper=1.6685 effort=0.583 velocity=2.09
- joint R_thumb_cmp_joint: limit lower=0 upper=0.96 effort=0.704 velocity=0 -> lower=0 upper=0.96 effort=0.704 velocity=2.09
- joint R_thumb_ip_joint: limit lower=0 upper=1.05 effort=0.182 velocity=0 -> lower=0 upper=1.05 effort=0.182 velocity=2.09
- joint R_thumb_mpp_joint: limit lower=0 upper=1.04 effort=0.632 velocity=0 -> lower=0 upper=1.04 effort=0.632 velocity=2.09

File: urdf/s2_v1_simple_clamp.urdf (robot description, URDF)
Before this commit: robot walker_s2_v1_simple_description, 35 links, 34 joints
Links:
- link L_hand_link: mass 0.28014837 -> 0.380120
- link R_hand_link: mass 0.28014837 -> 0.380120

File: urdf/s2_v1_simple_hand.urdf (robot description, URDF)
Before this commit: robot walker_s2_v1_simple_hand_description, 59 links, 58 joints
Links:
- link L_hand_base_link: mass 0 -> 0.169970
- link L_index_ip_link: mass 0.0133493 -> 0.01962738
- link L_index_mpp_link: mass 0.0147008 -> 0.02481999
- link L_little_ip_link: mass 0.0117927 -> 0.01658133
- link L_little_mpp_link: mass 0.0143021 -> 0.02481999
- link L_middle_ip_link: mass 0.0148881 -> 0.01962738
- link L_middle_mpp_link: mass 0.0143021 -> 0.02481999
- link L_palm_link: mass 0 -> 0.44979018
- link L_ring_ip_link: mass 0.0137479 -> 0.01962738
- link L_ring_mpp_link: mass 0.0143021 -> 0.02481999
- link L_thumb_cmp_link: mass 0.0151103 -> 0.01405089
- link L_thumb_ip_link: mass 0.0173112 -> 0.01901012
- link L_thumb_mpp_link: mass 0.067412 -> 0.09019498
- link R_hand_base_link: mass 0 -> 0.169970
- link R_index_ip_link: mass 0.0133493 -> 0.01962738
- link R_index_mpp_link: mass 0.0147008 -> 0.02481999
- link R_little_ip_link: mass 0.0117927 -> 0.01658133
- link R_little_mpp_link: mass 0.0143021 -> 0.02481999
- link R_middle_ip_link: mass 0.0148881 -> 0.01962738
- link R_middle_mpp_link: mass 0.0143021 -> 0.02481999
- link R_palm_link: mass 0 -> 0.44979018
- link R_ring_ip_link: mass 0.0137479 -> 0.01962738
- link R_ring_mpp_link: mass 0.0143021 -> 0.02481999
- link R_thumb_cmp_link: mass 0.0151103 -> 0.01405089
- link R_thumb_ip_link: mass 0.0173112 -> 0.01901012
- link R_thumb_mpp_link: mass 0.067412 -> 0.09019498
Joints:
- joint L_index_ip_joint: limit lower=0 upper=1.62 effort=0.311 velocity=0 -> lower=0 upper=1.62 effort=0.311 velocity=2.09
- joint L_index_mpp_joint: limit lower=0 upper=1.46 effort=0.583 velocity=0 -> lower=0 upper=1.6685 effort=0.583 velocity=2.09
- joint L_little_ip_joint: limit lower=0 upper=1.62 effort=0.257 velocity=0 -> lower=0 upper=1.62 effort=0.257 velocity=2.09
- joint L_little_mpp_joint: limit lower=0 upper=1.46 effort=0.528 velocity=0 -> lower=0 upper=1.6685 effort=0.528 velocity=2.09
- joint L_middle_ip_joint: limit lower=0 upper=1.62 effort=0.332 velocity=0 -> lower=0 upper=1.62 effort=0.332 velocity=2.09
- joint L_middle_mpp_joint: limit lower=0 upper=1.46 effort=0.604 velocity=0 -> lower=0 upper=1.6685 effort=0.604 velocity=2.09
- joint L_ring_ip_joint: limit lower=0 upper=1.62 effort=0.311 velocity=0 -> lower=0 upper=1.62 effort=0.311 velocity=2.09
- joint L_ring_mpp_joint: limit lower=0 upper=1.46 effort=0.583 velocity=0 -> lower=0 upper=1.6685 effort=0.583 velocity=2.09
- joint L_thumb_cmp_joint: limit lower=-0.96 upper=0 effort=0.704 velocity=0 -> lower=-0.96 upper=0 effort=0.704 velocity=2.09
- joint L_thumb_ip_joint: limit lower=0 upper=1.05 effort=0.182 velocity=0 -> lower=0 upper=1.05 effort=0.182 velocity=2.09
- joint L_thumb_mpp_joint: limit lower=0 upper=1.04 effort=0.632 velocity=0 -> lower=0 upper=1.04 effort=0.632 velocity=2.09
- joint R_index_ip_joint: limit lower=0 upper=1.62 effort=0.311 velocity=0 -> lower=0 upper=1.62 effort=0.311 velocity=2.09
- joint R_index_mpp_joint: limit lower=0 upper=1.46 effort=0.583 velocity=0 -> lower=0 upper=1.6685 effort=0.583 velocity=2.09
- joint R_little_ip_joint: limit lower=0 upper=1.62 effort=0.257 velocity=0 -> lower=0 upper=1.62 effort=0.257 velocity=2.09
- joint R_little_mpp_joint: limit lower=0 upper=1.46 effort=0.528 velocity=0 -> lower=0 upper=1.6685 effort=0.528 velocity=2.09
- joint R_middle_ip_joint: limit lower=0 upper=1.62 effort=0.332 velocity=0 -> lower=0 upper=1.62 effort=0.332 velocity=2.09
- joint R_middle_mpp_joint: limit lower=0 upper=1.46 effort=0.604 velocity=0 -> lower=0 upper=1.6685 effort=0.604 velocity=2.09
- joint R_ring_ip_joint: limit lower=0 upper=1.62 effort=0.311 velocity=0 -> lower=0 upper=1.62 effort=0.311 velocity=2.09
- joint R_ring_mpp_joint: limit lower=0 upper=1.46 effort=0.583 velocity=0 -> lower=0 upper=1.6685 effort=0.583 velocity=2.09
- joint R_thumb_cmp_joint: limit lower=0 upper=0.96 effort=0.704 velocity=0 -> lower=0 upper=0.96 effort=0.704 velocity=2.09
- joint R_thumb_ip_joint: limit lower=0 upper=1.05 effort=0.182 velocity=0 -> lower=0 upper=1.05 effort=0.182 velocity=2.09
- joint R_thumb_mpp_joint: limit lower=0 upper=1.04 effort=0.632 velocity=0 -> lower=0 upper=1.04 effort=0.632 velocity=2.09

Commit message: 重构执行器 mesh 目录结构，接入 v4 灵巧手与 v3 官方参数版，手部质量对齐官方规格
【网格重组】
- 将 34 个末端执行器 STL 从 s2_v1_simple/、s2_v1_complex/（各 67 个）中提取，
  按执行器类型与精度分为 9 个目录（共 180 STL，全部被引用、无孤儿）：
  * ee_gripper/            夹爪 6 个（simple/complex 共用，原两份字节级重复已去重）
  * ee_hand_v3_simple/     三代手 26 个（低精度，自官方手包补齐）
  * ee_hand_v3_complex/    三代手 26 个（高精度，与原 ee_hand_v3 相同）
  * ee_hand_v4_simple/     四代手 26 个（低精度，源自 ubt_hand_v4_evt3）
  * ee_hand_v4_complex/    四代手 26 个（高精度，源自 hand4_evt3complex）
  * ee_clamp_simple|complex/  夹板各 2 个（同一几何两种精度）
- 同步更新全部 URDF/MJCF 的 mesh 引用路径，simple 本体接 simple 执行器，
  complex 接 complex，精度档位严格匹配

【URDF 变更】（8 个 → 10 个）
- 删除旧的 v3 折叠版手部定义（官方包参数经 palm_joint 坐标折叠 + 整机团队
  质量口径 917.8g/手），替换为官方【三代手-URDF】参数版（palm_joint 带变换
  直通、官方限位 effort 1.35 N·m），零位指尖位置与旧版完全一致（偏差 0mm）
- 新增 v4 四代灵巧手（s2_v1_{simple,complex}_hand_v4.urdf），关节命名与 v3
  兼容；修正右腕挂接 180° 装配偏差（v4 右手为 Y 镜像约定，与整机 Z 180°
  约定不同，已按 Rz(π) 修正右腕挂接 rpy）

【MJCF 变更】（4 个 → 5 个）
- 删除旧的 s2_v1_simple_hand.xml（混合口径：折叠版 body 结构 + 整机团队
  限位/力矩）
- 新增 s2_v1_simple_hand_v3.xml / s2_v1_simple_hand_v4.xml，均从对应官方
  参数版 URDF 逐项转换生成：body 树与 URDF 同构（含 palm_joint 分层与
  v4 右腕修正）、关节限位与 actuatorfrcrange（±1.35 N·m）逐项一致、
  零位 FK 与 URDF 等价（偏差 <1μm）、52 motor、keyframe 59 qpos
- mesh 分别使用 ee_hand_v3_simple/ 与 ee_hand_v4_simple/

【质量对齐官方规格】
- v3 手部 26 link 质量与惯量等比缩放：645.84g → 单手精确 559g
- v4 手部 26 link 等比缩放：489.33g → 单手精确 815g（官方包仅建壳体）
- 质心位置不变，分布比例保留 CAD 口径；身体 33 link 未改动
- URDF（simple/complex 两版）与 MJCF（v3/v4 两版）全部同步，四份文件
  手部质量均精确命中官方规格

【文档】
- README.md：URDF 清单（10 个）、MJCF 清单（5 个）、mesh 目录说明、
  身体网格规模表（33 STL：simple 16 万面 7.8MB / complex 285 万面 136MB）、
  新增质量口径说明

【⚠ 不兼容变更】
- s2_v1_*_hand_v3.urdf 内容已替换为官方参数版（文件名不变）：
  * palm_link 坐标系语义改变：原与 hand_base_link 重合（挂接全零），现为
    掌部坐标系（偏移约 8.4cm + 大旋转）；外部代码的参考系请锚定
    hand_base_link / sixforce_link
  * 手部质量 917.8g → 559g，关节限位与力矩为官方口径（effort 1.35 N·m，
    mpp 限位 1.6685 → 1.46）
- mujoco/s2_v1_simple_hand.xml 已删除，拆分为 hand_v3 / hand_v4 两个文件，
  引用旧文件名的脚本需更新
- 旧 ee_hand_v3/ 目录已删除，路径引用需改为 ee_hand_v3_simple|complex/

File: urdf/s2_v1_complex_clamp.urdf (robot description, URDF)
Before this commit: robot walker_s2_v1_complex_description, 35 links, 34 joints
Links:
- link L_hand_link: geometry collision mesh filename=package://walker_s2_all/meshes/ee_clamp_complex/L_hand_link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; visual mesh filename=package://walker_s2_all/meshes/ee_clamp_complex/L_hand_link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
- link R_hand_link: geometry collision mesh filename=package://walker_s2_all/meshes/ee_clamp_complex/R_hand_link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; visual mesh filename=package://walker_s2_all/meshes/ee_clamp_complex/R_hand_link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

File: urdf/s2_v1_complex_gripper.urdf (robot description, URDF)
Before this commit: robot walker_s2_v1_complex_gripper_description, 39 links, 38 joints
Links:
- link L_gripper_base_link: geometry visual mesh filename=package://walker_s2_all/meshes/ee_gripper/L_gripper_base_li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
- link R_gripper_base_link: geometry visual mesh filename=package://walker_s2_all/meshes/ee_gripper/R_gripper_base_li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
- link left_L_gripper_link: geometry collision mesh filename=package://walker_s2_all/meshes/ee_gripper/left_L_gripper_li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; visual mesh filename=package://walker_s2_all/meshes/ee_gripper/left_L_gripper_li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
- link left_R_gripper_link: geometry collision mesh filename=package://walker_s2_all/meshes/ee_gripper/left_R_gripper_li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; visual mesh filename=package://walker_s2_all/meshes/ee_gripper/left_R_gripper_li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
- link right_L_gripper_link: geometry collision mesh filename=package://walker_s2_all/meshes/ee_gripper/right_L_gripper_l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; visual mesh filename=package://walker_s2_all/meshes/ee_gripper/right_L_gripper_l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
- link right_R_gripper_link: geometry collision mesh filename=package://walker_s2_all/meshes/ee_gripper/right_R_gripper_l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; visual mesh filename=package://walker_s2_all/meshes/ee_gripper/right_R_gripper_l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

File: urdf/s2_v1_simple_clamp.urdf (robot description, URDF)
Before this commit: robot walker_s2_v1_simple_description, 35 links, 34 joints
Links:
- link L_hand_link: geometry collision mesh filename=package://walker_s2_all/meshes/ee_clamp_simple/L_hand_link.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; visual mesh filename=package://walker_s2_all/meshes/ee_clamp_simple/L_hand_link.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
- link R_hand_link: geometry collision mesh filename=package://walker_s2_all/meshes/ee_clamp_simple/R_hand_link.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; visual mesh filename=package://walker_s2_all/meshes/ee_clamp_simple/R_hand_link.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

File: urdf/s2_v1_simple_gripper.urdf (robot description, URDF)
Before this commit: robot walker_s2_v1_simple_gripper_description, 39 links, 38 joints
Links:
- link L_gripper_base_link: geometry visual mesh filename=package://walker_s2_all/meshes/ee_gripper/L_gripper_base_li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
- link R_gripper_base_link: geometry visual mesh filename=package://walker_s2_all/meshes/ee_gripper/R_gripper_base_li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
- link left_L_gripper_link: geometry collision mesh filename=package://walker_s2_all/meshes/ee_gripper/left_L_gripper_li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; visual mesh filename=package://walker_s2_all/meshes/ee_gripper/left_L_gripper_li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
- link left_R_gripper_link: geometry collision mesh filename=package://walker_s2_all/meshes/ee_gripper/left_R_gripper_li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; visual mesh filename=package://walker_s2_all/meshes/ee_gripper/left_R_gripper_li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
- link right_L_gripper_link: geometry collision mesh filename=package://walker_s2_all/meshes/ee_gripper/right_L_gripper_l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; visual mesh filename=package://walker_s2_all/meshes/ee_gripper/right_L_gripper_l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
- link right_R_gripper_link: geometry collision mesh filename=package://walker_s2_all/meshes/ee_gripper/right_R_gripper_l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; visual mesh filename=package://walker_s2_all/meshes/ee_gripper/right_R_gripper_l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
